File: Automaattiaurinkopaneeli.kicad_pcb (KiCad board)
At the start: 2 copper layers, 39 parts, among them J1 Conn_02x04_Odd_Even, J10 Conn_01x16_Socket, J12 Conn_01x03_Socket, J13 Conn_01x05_Socket, J2 Conn_02x01, J3 Conn_01x02_Pin, J4 Conn_01x03_Pin, J5 Conn_01x03_Pin, J6 Conn_01x05_Pin, J7 Barrel_Jack_Switch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

Commit message: V0.6
Parts:
- added G***: LOGO, generic:fuuuuuuuuuuuuuuuuuuuuuuuuuuuuuuuuuuuuuuuuuuuuuuuuuuuuuuuuuuuuuuuuuuuuuuuuuuuuuuuuuuuuuuuuuuuuu, F.Cu at (195.5, 30.5)
- added REF**: Polarity_Center_Positive_6mm_SilkScreen, Symbol:Polarity_Center_Positive_6mm_SilkScreen, F.Cu at (147.0, 109.5)
- C1: footprint Capacitor_THT:C_Rect_L4.6mm_W4.6mm_P2.50mm_MKS02_FKP02 -> Capacitor_THT:C_Rect_L7.0mm_W3.5mm_P5.00mm
- RV1: footprint Potentiometer_THT:Potentiometer_Vishay_148-149_Single_Horizontal -> generic:Potentiometer_Generic_148-149_Single_Horizontal; moved to F.Cu
- U1: footprint RF_Module:ESP32-WROOM-32D -> generic:ESP32-WROOM-32D
- moved RV1 2.87 mm to (182.5, 94.5)
- renumbered J8 to 12V, J7 to 5V, J3 to RXTX1, J1 to Sensors1, J2 to flash1
Routing:
- net Net-(R10-Pad2): track 37.5 -> 28.7 mm
- net Net-(D2-A): track 459.4 -> 454.7 mm
- net Net-(R8-Pad1): track 81.3 -> 84.3 mm
- net Net-(D1-K): track 202.5 -> 204.0 mm
- net Net-(U2-VIOUT): track 47.4 -> 46.6 mm
Other:
- board outline added: 100.5 x 92 mm

Commit message: code
Parts:
- renumbered 12V to 12V1, 5V to J7
Connections:
- net Net-(D2-A) renamed GND
Routing:
- added copper zone on B.Cu, net GND
- added copper zone on F.Cu, net GND
Changed lines of the file:
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@@
 	)
 	(net 0 "")
-	(net 1 "Net-(D2-A)")
+	(net 1 "GND")
 	(net 2 "Net-(D1-K)")
 	(net 3 "Net-(U2-FILTER)")
@@
 			(layers "*.Cu" "*.Mask")
 			(remove_unused_layers no)
-			(net 1 "Net-(D2-A)")
+			(net 1 "GND")
 			(pintype "passive")
 		)
@@
 			(layers "*.Cu" "*.Mask")
 			(remove_unused_layers no)
-			(net 1 "Net-(D2-A)")
+			(net 1 "GND")
 			(pinfunction "Pin_1")
 			(pintype "passive")
@@
 			(layers "*.Cu" "*.Mask")
 			(remove_unused_layers no)
-			(net 1 "Net-(D2-A)")
+			(net 1 "GND")
 			(pinfunction "GND")
 			(pintype "power_in")
@@
 			(layers "*.Cu" "*.Mask")
 			(remove_unused_layers no)
-			(net 1 "Net-(D2-A)")
+			(net 1 "GND")
 			(pinfunction "Pin_1")
 			(pintype "passive")
@@
 			(layers "*.Cu" "*.Mask")
 			(remove_unused_layers no)
-			(net 1 "Net-(D2-A)")
+			(net 1 "GND")
 			(pinfunction "Pin_2")
 			(pintype "passive")
@@
 			(layers "*.Cu" "*.Mask")
 			(remove_unused_layers no)
-			(net 1 "Net-(D2-A)")
+			(net 1 "GND")
 			(pinfunction "Pin_5")
 			(pintype "passive")
@@
 		(descr "Wuerth electronics barrel jack connector (5.5mm outher diameter, inner diameter 2.05mm or 2.55mm depending on exact order number), See: http://katalog.we-online.de/em/datasheet/6941xx301002.pdf")
 		(tags "connector barrel jack")
-		(property "Reference" "5V"
+		(property "Reference" "J7"
 			(at 0 -2.5 0)
 			(layer "F.SilkS")
@@
 			(layers "*.Cu" "*.Mask")
 			(remove_unused_layers no)
-			(net 1 "Net-(D2-A)")
+			(net 1 "GND")
 			(pintype "passive")
 		)
@@
 			(layers "*.Cu" "*.Mask")
 			(remove_unused_layers no)
-			(net 1 "Net-(D2-A)")
+			(net 1 "GND")
 			(pintype "passive")
 		)
@@
 			(layers "*.Cu" "*.Mask")
 			(remove_unused_layers no)
-			(net 1 "Net-(D2-A)")
+			(net 1 "GND")
 			(pintype "passive")
 		)
@@
 			(layers "*.Cu" "*.Mask")
 			(remove_unused_layers no)
-			(net 1 "Net-(D2-A)")
+			(net 1 "GND")
 			(pintype "passive")
 		)
@@
 			(layers "*.Cu" "*.Mask")
 			(remove_unused_layers no)
-			(net 1 "Net-(D2-A)")
+			(net 1 "GND")
 			(pintype "passive")
 		)
@@
 			(layers "*.Cu" "*.Mask")
 			(remove_unused_layers no)
-			(net 1 "Net-(D2-A)")
+			(net 1 "GND")
 			(pintype "passive")
 		)
@@
 			(layers "*.Cu" "*.Mask")
 			(remove_unused_layers no)
-			(net 1 "Net-(D2-A)")
+			(net 1 "GND")
 			(pintype "passive")
 		)
@@
 			(layers "*.Cu" "*.Mask")
 			(remove_unused_layers no)
-			(net 1 "Net-(D2-A)")
+			(net 1 "GND")
 			(pintype "passive")
 		)
@@
 			(layers "*.Cu" "*.Mask")
 			(remove_unused_layers no)
-			(net 1 "Net-(D2-A)")
+			(net 1 "GND")
 			(pintype "passive")
 		)
@@
 			(layers "*.Cu" "*.Mask")
 			(remove_unused_layers no)
-			(net 1 "Net-(D2-A)")
+			(net 1 "GND")
 			(pintype "passive")
 		)
@@
 			(layers "*.Cu" "*.Mask")
 			(remove_unused_layers no)
-			(net 1 "Net-(D2-A)")
+			(net 1 "GND")
 			(pintype "passive")
 		)
@@
 			(layers "*.Cu" "*.Mask")
 			(remove_unused_layers no)
-			(net 1 "Net-(D2-A)")
+			(net 1 "GND")
 			(pinfunction "A")
 			(pintype "passive")
@@
 			(layers "*.Cu" "*.Mask")
 			(remove_unused_layers no)
-			(net 1 "Net-(D2-A)")
+			(net 1 "GND")
 			(pinfunction "Pin_1")
 			(pintype "passive")
@@
 			(layers "*.Cu" "*.Mask")
 			(remove_unused_layers no)
-			(net 1 "Net-(D2-A)")
+			(net 1 "GND")
 			(pintype "passive")
 		)
@@
 			(layers "*.Cu" "*.Mask")
 			(remove_unused_layers no)
-			(net 1 "Net-(D2-A)")
+			(net 1 "GND")
 			(pintype "passive")
 		)
@@
 			(layers "*.Cu" "*.Mask")
 			(remove_unused_layers no)
-			(net 1 "Net-(D2-A)")
+			(net 1 "GND")
 			(pintype "passive")
 		)
@@
 		(descr "Through hole straight pin header, 1x02, 2.54mm pitch, single row")
 		(tags "Through hole pin header THT 1x02 2.54mm single row")
-		(property "Reference" "12V"
+		(property "Reference" "12V1"
 			(at -1 -3.225 180)
 			(layer "F.SilkS")
@@
 			(layers "*.Cu" "*.Mask")
 			(remove_unused_layers no)
-			(net 1 "Net-(D2-A)")
+			(net 1 "GND")
 			(pintype "passive")
 		)
@@
 			(layers "*.Cu" "*.Mask")
 			(remove_unused_layers no)
-			(net 1 "Net-(D2-A)")
+			(net 1 "GND")
 			(pintype "passive")
 		)
@@
 			(layers "*.Cu" "*.Mask")
 			(remove_unused_layers no)
-			(net 1 "Net-(D2-A)")
+			(net 1 "GND")
 			(pinfunction "Pin_1")
 			(pintype "passive")
@@
 			(layers "*.Cu" "*.Mask")
 			(remove_unused_layers no)
-			(net 1 "Net-(D2-A)")
+			(net 1 "GND")
 			(pinfunction "Pin_5")
 			(pintype "passive")
@@
 			(layers "*.Cu" "*.Mask")
 			(remove_unused_layers no)
-			(net 1 "Net-(D2-A)")
+			(net 1 "GND")
 			(pinfunction "Pin_16")
 			(pintype "passive")
@@
 			(layers "*.Cu" "*.Mask")
 			(remove_unused_layers no)
-			(net 1 "Net-(D2-A)")
+			(net 1 "GND")
 			(pintype "passive")
 		)
@@
 			(layers "*.Cu" "*.Mask")
 			(remove_unused_layers no)
-			(net 1 "Net-(D2-A)")
+			(net 1 "GND")
 			(pintype "passive")
 		)
@@
 			(layers "*.Cu" "*.Mask")
 			(remove_unused_layers no)
-			(net 1 "Net-(D2-A)")
+			(net 1 "GND")
 			(pintype "passive")
 		)
@@
 			(layers "B.Cu" "B.Paste" "B.Mask")
 			(roundrect_rratio 0.25)
-			(net 1 "Net-(D2-A)")
+			(net 1 "GND")
 			(pinfunction "GND")
 			(pintype "power_in")
@@
 			(size 1.5 0.9)
 			(layers "B.Cu" "B.Paste" "B.Mask")
-			(net 1 "Net-(D2-A)")
+			(net 1 "GND")
 			(pinfunction "GND")
 			(pintype "power_in")
@@
 			(size 1.5 0.9)
 			(layers "B.Cu" "B.Paste" "B.Mask")
-			(net 1 "Net-(D2-A)")
+			(net 1 "GND")
 			(pinfunction "GND")
 			(pintype "passive")
@@
 			(size 1.5 0.9)
 			(layers "B.Cu" "B.Paste" "B.Mask")
-			(net 1 "Net-(D2-A)")
+			(net 1 "GND")
 			(pinfunction "GND")
 			(pintype "passive")
@@
 			(size 0.9 0.9)
 			(layers "B.Cu" "B.Paste")
-			(net 1 "Net-(D2-A)")
+			(net 1 "GND")
 			(pinfunction "GND")
 			(pintype "passive")
@@
 			(size 0.9 0.9)
 			(layers "B.Cu" "B.Paste")
-			(net 1 "Net-(D2-A)")
+			(net 1 "GND")
 			(pinfunction "GND")
 			(pintype "passive")
@@
 			(size 0.9 0.9)
 			(layers "B.Cu" "B.Paste")
-			(net 1 "Net-(D2-A)")
+			(net 1 "GND")
 			(pinfunction "GND")
 			(pintype "passive")
@@
 			(layers "*.Cu" "*.Mask")
 			(remove_unused_layers no)
-			(net 1 "Net-(D2-A)")
+			(net 1 "GND")
 			(pinfunction "GND")
 			(pintype "passive")
@@
 			(layers "*.Cu" "*.Mask")
 			(remove_unused_layers no)
-			(net 1 "Net-(D2-A)")
+			(net 1 "GND")
 			(pinfunction "GND")
 			(pintype "passive")
@@
 			(size 0.9 0.9)
 			(layers "B.Cu" "B.Paste")
-			(net 1 "Net-(D2-A)")
+			(net 1 "GND")
 			(pinfunction "GND")
 			(pintype "passive")
@@
 			(size 0.9 0.9)
 			(layers "B.Cu" "B.Paste")
-			(net 1 "Net-(D2-A)")
+			(net 1 "GND")
 			(pinfunction "GND")
 			(pintype "passive")
@@
 			(size 3.8 3.8)
 			(layers "B.Cu" "B.Mask")
-			(net 1 "Net-(D2-A)")
+			(net 1 "GND")
 			(pinfunction "GND")
 			(pintype "passive")
@@
 			(size 0.9 0.9)
 			(layers "B.Cu" "B.Paste")
-			(net 1 "Net-(D2-A)")
+			(net 1 "GND")
 			(pinfunction "GND")
 			(pintype "passive")
@@
 			(layers "*.Cu" "*.Mask")
 			(remove_unused_layers no)
-			(net 1 "Net-(D2-A)")
+			(net 1 "GND")
 			(pinfunction "GND")
 			(pintype "passive")
@@
 			(layers "*.Cu" "*.Mask")
 			(remove_unused_layers no)
-			(net 1 "Net-(D2-A)")
+			(net 1 "GND")
 			(pinfunction "GND")
 			(pintype "passive")
@@
 			(size 0.9 0.9)
 			(layers "B.Cu" "B.Paste")
-			(net 1 "Net-(D2-A)")
+			(net 1 "GND")
 			(pinfunction "GND")
 			(pintype "passive")
@@
 			(size 0.9 0.9)
 			(layers "B.Cu" "B.Paste")
-			(net 1 "Net-(D2-A)")
+			(net 1 "GND")
 			(pinfunction "GND")
 			(pintype "passive")
@@
 			(size 0.9 0.9)
 			(layers "B.Cu" "B.Paste")
-			(net 1 "Net-(D2-A)")
+			(net 1 "GND")
 			(pinfunction "GND")
 			(pintype "passive")
@@
 		(net 50)
 	)
+	(zone
+		(net 1)
+		(net_name "GND")
+		(layer "F.Cu")
+		(hatch edge 0.5)
+		(connect_pads
+			(clearance 0.5)
+		)
+		(min_thickness 0.25)
+		(filled_areas_thickness no)
+		(fill yes
+			(thermal_gap 0.5)
+			(thermal_bridge_width 0.5)
+		)
+		(polygon
+			(pts
+				(xy 107 113) (xy 107 21) (xy 207.5 21) (xy 207.5 113)
+			)
+		)
+	)
+	(zone
+		(net 1)
+		(net_name "GND")
+		(layer "B.Cu")
+		(hatch edge 0.5)
+		(priority 1)
+		(connect_pads
+			(clearance 0.5)
+		)
+		(min_thickness 0.25)
+		(filled_areas_thickness no)
+		(fill yes
+			(thermal_gap 0.5)
+			(thermal_bridge_width 0.5)
+		)
+		(polygon
+			(pts
+				(xy 107 21) (xy 207.5 21) (xy 207.5 113) (xy 107 113)
+			)
+		)
+	)
 )
